File: VoyagerSplitKicad/VoyagerSplitKicad.kicad_sch (KiCad schematic)
At the start: 3 parts

Commit message: layed out one half of pcb
Parts:
- H11, H12, H13: footprint (none) -> Panelization:MouseBite-Slot_2.0x4.5mm_outset_D0.5mm_P0.85mm_7h
Changed lines of the file:
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@@
 			)
 		)
-		(property "Footprint" ""
+		(property "Footprint" "Panelization:MouseBite-Slot_2.0x4.5mm_outset_D0.5mm_P0.85mm_7h"
 			(at 88.9 27.94 0)
 			(effects
@@
 			)
 		)
-		(property "Footprint" ""
+		(property "Footprint" "Panelization:MouseBite-Slot_2.0x4.5mm_outset_D0.5mm_P0.85mm_7h"
 			(at 88.9 34.29 0)
 			(effects
@@
 			)
 		)
-		(property "Footprint" ""
+		(property "Footprint" "Panelization:MouseBite-Slot_2.0x4.5mm_outset_D0.5mm_P0.85mm_7h"
 			(at 88.9 40.64 0)
 			(effects
