File: VoyagerSplitKicad/VoyagerSplitKicad.kicad_pcb (KiCad board)
At the start: 2 copper layers, 6.5 x 2 mm, 131 parts, among them SW1 SW_Push, SW10 SW_Push, SW11 SW_Push, SW12 SW_Push, SW13 SW_Push, SW14 SW_Push, SW15 SW_Push, SW16 SW_Push, SW17 SW_Push, SW18 SW_Push, SW19 SW_Push, SW2 SW_Push, SW20 SW_Push, SW21 SW_Push, SW22 SW_Push, SW23 SW_Push, SW24 SW_Push, SW25 SW_Push, SW26 SW_Push, SW27 SW_Push, SW28 SW_Push, SW29 SW_Push, SW3 SW_Push, SW30 SW_Push, SW31 SW_Push, SW32 SW_Push, SW33 SW_Push, SW34 SW_Push, SW35 SW_Push, SW36 SW_Push, SW37 SW_Push, SW38 SW_Push, SW39 SW_Push, SW4 SW_Push, SW40 SW_Push, SW41 SW_Push, SW42 SW_Push, SW43 SW_Push, SW44 SW_Push, SW45 SW_Push, SW46 SW_Push, SW47 SW_Push, SW48 SW_Push, SW5 SW_Push, SW51 SW_Push, SW52 SW_Push, SW53 SW_Push, SW54 SW_Push, SW57 SW_Push, SW58 SW_Push, SW59 SW_Push, SW6 SW_Push, SW60 SW_Push, SW7 SW_Push, SW8 SW_Push, SW9 SW_Push, U1 XIAO-nRF52840-SMD, U2 XIAO-nRF52840-SMD

Commit message: laying out 2nd half of PCB and getting edge cut
Parts:
- D13, D14, D15, D16, D2, D25, D26, D27, D28, D29, D30, D31, D32, D4, D41, D42, D43, D44, D45, D46, D47, D48, D57, D58, D59, D60, D7, D8, SW13, SW14, SW15, SW16, SW2, SW25, SW26, SW27, SW28, SW29, SW30, SW31, SW32, SW4, SW41, SW42, SW43, SW44, SW45, SW46, SW47, SW48, SW57, SW58, SW59, SW60, SW7, SW8, TP2, TP4, U2: moved to B.Cu
- H1, H10, H2, H3, H4, H5, H6, H7, H8, H9: footprint MountingHole:MountingHole_3.2mm_M3 -> MountingHole:MountingHole_2.2mm_M2
- moved D60 215.3 mm to (72.1, 167.4), turned to 120 degrees
- moved D59 214.5 mm to (80.6, 182.2), turned to 120 degrees
- moved H8 206.7 mm to (67.8, 150.9)
- moved D58 197.1 mm to (98.9, 176.8), turned to 90 degrees
- moved U2 189.1 mm to (75.7, 137.7), turned to 180 degrees
- moved H10 187.6 mm to (92.0, 165.3)
- moved D48 185.7 mm to (90.0, 158.1), turned to 90 degrees
- moved H1 184.3 mm to (302.8, 165.4)
- moved H7 183.4 mm to (326.8, 151.0)
- moved D47 182.4 mm to (90.0, 141.1), turned to 90 degrees
- moved D57 182.1 mm to (116.9, 175.1), turned to 90 degrees
- moved D52 181.2 mm to (284.5, 176.8)
- moved D1 181.2 mm to (203.5, 108.8)
- moved D10 181.2 mm to (203.5, 159.8)
- moved D11 181.2 mm to (221.5, 142.8)
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Other:
- board size 6.5 x 2 mm -> 274.6 x 100.5 mm

Commit message: added 3d
Parts:
- H1, H10, H2, H3, H4, H5, H6, H7, H8, H9: footprint MountingHole:MountingHole_2.2mm_M2 -> CustomMousebite:MountingHole_2.2mm_M2
- H11, H12, H13: footprint Panelization:MouseBite-Slot_2.0x4.5mm_outset_D0.5mm_P0.85mm_7h -> CustomMousebite:MouseBite-Slot_2.0x4.5mm_outset_D0.5mm_P0.85mm_7h
- moved TP3 6.85 mm to (312.6, 151.3)
- moved TP2 6.77 mm to (84.6, 157.8)
- moved TP4 4.35 mm to (84.6, 152.0)
- moved TP1 3.72 mm to (311.1, 156.1)
- moved H6 0.80 mm to (126.4, 159.6)
- moved H10 0.60 mm to (91.4, 165.3)
- moved U2 0.46 mm to (76.2, 137.7)
- moved SW59 0.45 mm to (82.3, 174.8)
- moved D59 0.45 mm to (80.2, 182.0)
- moved D60 0.45 mm to (71.7, 167.2)
- moved SW60 0.45 mm to (73.8, 160.1)
- moved D1 0.40 mm to (203.9, 108.7)
- moved D10 0.40 mm to (203.9, 159.7)
- moved D11 0.40 mm to (221.9, 142.7)
- moved D12 0.40 mm to (221.9, 159.7)
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Routing:
- net /left/COL2: track 0.00 -> 207.0 mm, vias 0 -> 3
- net /left/COL0: track 0.00 -> 180.2 mm, vias 0 -> 1
- net /left/COL1: track 0.00 -> 176.9 mm, vias 0 -> 1
- net /right/COL0: track 0.00 -> 168.6 mm, vias 0 -> 1
- net /left/COL4: track 0.00 -> 160.0 mm, vias 0 -> 5
- net /left/COL5: track 0.00 -> 151.6 mm
- net /right/COL1: track 0.00 -> 147.3 mm, vias 0 -> 1
- net /right/COL2: track 0.00 -> 146.4 mm, vias 0 -> 1
- net /right/ROW0: track 0.00 -> 137.3 mm, vias 0 -> 12
- net /left/COL3: track 0.00 -> 135.4 mm, vias 0 -> 3
- net /left/ROW0: track 0.00 -> 135.3 mm, vias 0 -> 12
- net /right/COL3: track 0.00 -> 129.8 mm, vias 0 -> 1
- net /right/COL4: track 0.00 -> 128.1 mm, vias 0 -> 1
- net /right/ROW3: track 0.00 -> 124.4 mm, vias 0 -> 9
- net /right/ROW1: track 0.00 -> 123.2 mm, vias 0 -> 12
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
Commit message: flipped xiao
Parts:
- U1, U2: moved to F.Cu
- turned U1 to 0 degrees
- turned U2 to 0 degrees
Routing:
- net /right/COL2: track 146.4 -> 182.8 mm, vias 1 -> 0
- net /left/COL1: track 176.9 -> 154.3 mm, vias 1 -> 0
- net /left/COL0: track 180.2 -> 158.3 mm, vias 1 -> 0
- net /right/COL1: track 147.3 -> 169.2 mm, vias 1 -> 0
- net /left/ROW2: track 110.5 -> 130.4 mm, vias 12 -> 11
- net /left/ROW1: track 119.6 -> 138.4 mm, vias 12 -> 11
- net /left/COL2: track 207.0 -> 188.6 mm, vias 3 -> 2
- net /right/COL0: track 168.6 -> 186.0 mm, vias 1 -> 0
- net /right/ROW2: track 115.5 -> 100.3 mm, vias 12 -> 11
- net /left/ROW3: track 119.0 -> 133.9 mm, vias 2 -> 1
- net /right/COL3: track 129.8 -> 143.1 mm, vias 1 -> 0
- net /right/ROW3: track 124.4 -> 113.4 mm
- net /right/ROW0: track 137.3 -> 126.9 mm, vias 12 -> 11
- net /right/ROW1: track 123.2 -> 112.9 mm, vias 12 -> 11
- net /left/COL5: track 151.6 -> 142.6 mm, vias 0 -> 1
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
Commit message: CAD!
Parts:
- +: renamed from TP2; moved to F.Cu
- +: renamed from TP1; moved to F.Cu
- -: renamed from TP4; moved to F.Cu
- -: renamed from TP3; moved to F.Cu
- moved D32 1.65 mm to (126.0, 154.7)
- turned + to 0 degrees (x2)
- turned - to 0 degrees (x2)
Routing:
- net /right/COL3: track 143.1 -> 145.8 mm
- net /right/ROW3: track 113.4 -> 111.3 mm
- net /left/VBAT: track 19.5 -> 19.6 mm, vias 0 -> 1
- net GND: vias 1 -> 2
